File: kicad_docs/2164_phasor_plug_in_board.sch (KiCad schematic (older format))
At the start: 85 parts, among them J1 Conn_01x04_Male, J2 Conn_01x04_Male, J3 Conn_01x04_Male, J4 Conn_01x08_Male, U1 TL074, U2 SSM2164, U3 TL074, U4 SSM2164, U5 TL074, U6 TL072

Commit message: change trimmers to cheaper TH type
Parts:
- RV1, RV2, RV3: footprint Potentiometer_SMD:Potentiometer_Bourns_3269W_Vertical -> Potentiometer_THT:Potentiometer_Bourns_3296W_Vertical
- U2, U4: symbol jordans_parts:SSM2164 -> 2164_phasor_plug_in_board-rescue:SSM2164-jordans_parts
Connections:
- net at J4.3 (Pin_3), J4.4 (Pin_4): now also RV3.3; no longer RV3.1
- net at R40.2, RV3.2: now also RV3.1; no longer RV3.3
Changed lines of the file:
@@
 F 0 "RV1" H 3100 10400 50  0000 R CNN
 F 1 "10k" V 3150 10450 50  0000 R CNN
-F 2 "Potentiometer_SMD:Potentiometer_Bourns_3269W_Vertical" H 3150 10400 50  0001 C CNN
+F 2 "Potentiometer_THT:Potentiometer_Bourns_3296W_Vertical" H 3150 10400 50  0001 C CNN
 F 3 "~" H 3150 10400 50  0001 C CNN
 	1    3150 10400
@@
 F 0 "RV2" V 3385 11200 50  0000 C CNN
 F 1 "100k" V 3500 11200 50  0000 C CNN
-F 2 "Potentiometer_SMD:Potentiometer_Bourns_3269W_Vertical" H 3500 11200 50  0001 C CNN
+F 2 "Potentiometer_THT:Potentiometer_Bourns_3296W_Vertical" H 3500 11200 50  0001 C CNN
 F 3 "~" H 3500 11200 50  0001 C CNN
 	1    3500 11200
@@
 	2750 5600 2750 5700
 $Comp
-L jordans_parts:SSM2164 U2
+L 2164_phasor_plug_in_board-rescue:SSM2164-jordans_parts U2
 U 1 1 5CF83552
 P 2250 5400
@@
 	5250 5600 5250 5700
 $Comp
-L jordans_parts:SSM2164 U2
+L 2164_phasor_plug_in_board-rescue:SSM2164-jordans_parts U2
 U 2 1 5D88BF62
 P 4750 5400
@@
 	9200 5600 9200 5700
 $Comp
-L jordans_parts:SSM2164 U2
+L 2164_phasor_plug_in_board-rescue:SSM2164-jordans_parts U2
 U 3 1 5E0F7FF8
 P 8700 5400
@@
 	11700 5600 11700 5700
 $Comp
-L jordans_parts:SSM2164 U2
+L 2164_phasor_plug_in_board-rescue:SSM2164-jordans_parts U2
 U 4 1 5E0F8074
 P 11200 5400
@@
 	15650 5650 15650 5750
 $Comp
-L jordans_parts:SSM2164 U4
+L 2164_phasor_plug_in_board-rescue:SSM2164-jordans_parts U4
 U 1 1 5E1E05C4
 P 16100 9800
@@
 	18150 5650 18150 5750
 $Comp
-L jordans_parts:SSM2164 U4
+L 2164_phasor_plug_in_board-rescue:SSM2164-jordans_parts U4
 U 2 1 5E1E0640
 P 16100 8100
@@
 Fcv
 $Comp
-L jordans_parts:SSM2164 U4
+L 2164_phasor_plug_in_board-rescue:SSM2164-jordans_parts U4
 U 4 1 5E502D3D
 P 15150 5450
@@
 Connection ~ 17500 10550
 $Comp
-L jordans_parts:SSM2164 U4
+L 2164_phasor_plug_in_board-rescue:SSM2164-jordans_parts U4
 U 3 1 5CF8623C
 P 17650 5450
@@
 F 0 "RV3" V 18135 10550 50  0000 C CNN
 F 1 "100k" V 18250 10550 50  0000 C CNN
-F 2 "Potentiometer_SMD:Potentiometer_Bourns_3269W_Vertical" H 18250 10550 50  0001 C CNN
+F 2 "Potentiometer_THT:Potentiometer_Bourns_3296W_Vertical" H 18250 10550 50  0001 C CNN
 F 3 "~" H 18250 10550 50  0001 C CNN
 	1    18250 10550
-	0    1    -1   0
+	0    -1   -1   0
 $EndComp
 $Comp
@@
 $EndComp
 $Comp
-L jordans_parts:SSM2164 U4
+L 2164_phasor_plug_in_board-rescue:SSM2164-jordans_parts U4
 U 5 1 5F0E7D6D
 P 10850 15150
@@
 	10700 15350 10800 15350
 $Comp
-L jordans_parts:SSM2164 U2
+L 2164_phasor_plug_in_board-rescue:SSM2164-jordans_parts U2
 U 5 1 5F903A8D
 P 10050 15150
